Commit message: min

File: Project_2/src/pet_robot/urdf/wooden_robot_edited.xacro (robot description, xacro)
@@ -1,4 +1,13 @@
 <?xml version='1.0'?>
 <robot name="wooden_robot" xmlns:xacro="http://www.ros.org/wiki/xacro">
+  <material name="blue">
+       <color rgba="0 0 0.8 1"/>
+  </material>
+  <material name="white">
+        <color rgba="0 0 0 1"/>
+  </material>
+  <gazebo reference="chassis">
+   <material>Gazebo/Blue</material>
+  </gazebo>
   <xacro:include filename="$(find pet_robot)/urdf/pet_robot.gazebo" />
   <link name="robot_footprint"></link>
@@ -30,4 +39,5 @@
         <box size=".4 .2 .1"/>
       </geometry>
+      <material name="orange"/>
     </visual>
     <collision name='back_caster_collision'>
@@ -42,4 +52,5 @@
         <sphere radius="0.05"/>
       </geometry>
+      <material name="blue"/>
     </visual>
     <collision name='front_caster_collision'>
@@ -54,4 +65,5 @@
         <sphere radius="0.05"/>
       </geometry>
+      <material name="blue"/>
     </visual>
   </link>
@@ -78,4 +90,5 @@
       </geometry>
     </visual>
+    <material name="blue"/>
   </link>
 <link name='right_wheel'>
@@ -101,4 +114,5 @@
       </geometry>
     </visual>
+    <material name="blue"/>
   </link>
   <link name='camera'>
